File: kicad/kicad.kicad_sch (KiCad schematic)
At the start: 10 parts, among them J1 switch, SW2 button, SW3 button, SW4 button, U1 ESP-12F, U2 AMS1117-3.3

Commit message: updated frontend backend, improved cpp, added admin panel
Parts:
- removed J1: switch, Connector_PinHeader_2.00mm:PinHeader_2x03_P2.00mm_Vertical_SMD, symbol Connector_Generic:Conn_02x03_Row_Letter_First
- removed SW2, SW3, SW4: button, Button_Switch_THT:SW_PUSH_6mm_H4.3mm, symbol Switch:SW_Push
- added ADC1, GND1, GND2, SCL1, SDA1, VCC1, VCC2: OUT, TestPoint:TestPoint_Pad_2.0x2.0mm, symbol Mechanical:MountingHole_Pad
- added C1: 10V 1000UF, Capacitor_THT:CP_Radial_D8.0mm_P3.80mm, symbol Device:C_Polarized
- added C2: 10v 47UF, Capacitor_THT:CP_Radial_D4.0mm_P1.50mm, symbol Device:C_Polarized
- added D1, D2: LED, LED_THT:LED_D5.0mm, symbol Device:LED
- added J1: Boot Switch, Connector_PinHeader_2.54mm:PinHeader_2x03_P2.54mm_Vertical_SMD, symbol Connector_Generic:Conn_02x03_Top_Bottom
- added J2: input, Connector_PinHeader_2.54mm:PinHeader_2x05_P2.54mm_Vertical_SMD, symbol Connector_Generic:Conn_02x05_Odd_Even
- added R5: 200, Resistor_SMD:R_2512_6332Metric_Pad1.40x3.35mm_HandSolder, symbol Device:R
- added R6, R7: idk, Resistor_SMD:R_2512_6332Metric_Pad1.40x3.35mm_HandSolder, symbol Device:R
- added R8: 10k, Resistor_SMD:R_2512_6332Metric_Pad1.40x3.35mm_HandSolder, symbol Device:R
- R3: value 220 -> 10k
- R4: value 100 -> 200
Connections:
- net GND is gone; now on net -BATT: R4.1, U1.15 (GND), U2.1 (GND)
- net RESET: now also J2.1 (Pin_1), J2.10 (Pin_10)
- net RX: now also J2.5 (Pin_5), J2.6 (Pin_6)
- net TX: now also J2.3 (Pin_3), J2.8 (Pin_8)
- net -BATT: now reaches R2.2
- net -BATT: now also C1.2, C2.2, GND1.1, GND2.1, J1.2 (Pin_2), J1.3 (Pin_3), J1.5 (Pin_5), J1.6 (Pin_6), J2.2 (Pin_2), J2.9 (Pin_9), R5.1, R7.2
- net at R1.1: now also U1.8 (VCC), U2.2 (VO), C2.1, VCC1.1, VCC2.1; no longer U1.3 (EN)
- net at U1.6 (GPIO12): now also D1.1 (K)
- net at U1.7 (GPIO13): now also D2.1 (K)
- net ADC: no longer names the net of R3.1
- net ADC: now also J1.1 (Pin_1), J1.4 (Pin_4)
- net IO 0: no longer names the net of U1.18 (GPIO0)
- net IO 0: now also R3.2
- net SCL: no longer names the net of U1.5 (GPIO14)
- net SCL: now also SCL1.1
- net SDA: no longer names the net of U1.17 (GPIO2)
- net SDA: now also SDA1.1
- net SIG: no longer names the net of U1.12 (GPIO10)
- net SIG: now also R8.2
- removed net VCC: R1.2, U1.8 (VCC), U2.2 (VO)
- net VIN renamed +BATT
- net +BATT: now also C1.1, J2.4 (Pin_4), J2.7 (Pin_7), R6.1
- new net: D2.2 (A), R5.2
- new net: D1.2 (A), R4.2
- new net: R6.2, R7.1, R8.1
- new net: ADC1.1, U1.2 (ADC)
- new net: R1.2, U1.3 (EN)
- no-connect marks 7 -> 8
Other:
- note removed: "BATTERY"
- note removed: "PROGRAMMING INTERFACE"
- moved on the sheet: R1, R2, U1, U2
